File: PCB/PMSA+SHT31_board/SHT31.brd (EAGLE design)
At the start: 41.7 x 49.2 mm, 8 parts, among them CN2 CON_PINHD-2X15, U2 SHT31-DIS

Commit message: insertion NOX & CO Captor
Parts:
- moved CN2 0.46 mm to (18.7, 43.2)
- moved U$9 0.25 mm to (30.7, 5.69)
Connections:
- removed net ALERT: U2.3
Routing:
- net GND: track 107.9 -> 102.3 mm
- net PT_RX: track 60.8 -> 65.2 mm, vias 0 -> 2
- net VDD: track 71.8 -> 74.8 mm
- net PT_TX: track 73.2 -> 70.9 mm
Other:
- outline, holes or cut-outs redrawn
