File: source file/gas sensor/SensorBoard.sch (EAGLE design)
At the start: 18 parts, among them CN2 CON_PINHD-2X15, Q3 MOSFET-NCHANNELBSS138, U2 SHT31-DIS, U3 MICS-4514

Commit message: insertion NOX & CO Captor
Parts:
- removed C2: 10uF, microbuilder:CAP_CERAMIC_1206
- removed CN2: CON_PINHD-2X15, akita:CON_PINHD-2X15
- removed R6, R7, R8, R9: 10K, microbuilder:RESISTOR_1206MP
- removed U$9: PLANTOWER, Airbeam:PLANTOWER
- removed U2: SHT31-DIS, microbuilder:SHT3X
- C13: device SparkFun-Capacitors:CAP0805 -> SparkFun-Capacitors:CAP1206
- R13: device SparkFun-Resistors:RESISTOR0603 -> SparkFun-Resistors:RESISTOR1206
- R19, R21: device SparkFun-Resistors:RESISTOR0805-RES -> SparkFun-Resistors:RESISTOR1206
Connections:
- removed net ADDR: R8.1, U2.ADDR
- removed net ALERT: U2.ALERT
- removed net PT_RST: U$9.RST
- removed net PT_RX: CN2.3, U$9.RX
- removed net PT_TX: CN2.1, R17.1, U$9.TX
- removed net RST: R9.2, U2.NRESET
- removed net SCL: CN2.18, R6.1, U2.SCL
- removed net SDA: CN2.17, R7.1, U2.SDA
- removed net SLEEP_PT: U$9.SET
- removed net VDD: C13.1, C2.1, CN2.27, R6.2, R7.2, R9.1, U$9.VCC, U$9.\VCC, U2.VDD, U3.RH2_OX, U3.RH2_RED, U3.RS2_OX, U3.RS2_RED
- new net 3V3: C13.1, U3.RH2_OX, U3.RH2_RED, U3.RS2_OX, U3.RS2_RED
- new net PRE: R17.1
- net GND: no longer C2.2, CN2.2, R8.2, U$9.GND, U$9.\GND, U2.R(VSS), U2.VSS
- net VNOX: no longer CN2.19
- net VRED: no longer CN2.20
Other:
- note removed: "Plantower"
- note removed: "RST -> Pin 7"
- note removed: "RX -> Pin 6"
- note removed: "SHT31"
- note removed: "SLEEP -> Pin 1"
- note removed: "TX -> Pin 12"
