File: PCB/aircitizen-m5stack-v2/aircitizen-m5stack-v2.brd (EAGLE design)
At the start: 41.7 x 49.2 mm, 18 parts, among them CN2 CON_PINHD-2X15, Q3 MOSFET-NCHANNELBSS138, U2 SHT31-DIS, U3 MICS-4514

Commit message: Nouvel version pcb V2
Parts:
- removed C2: 10uF, microbuilder:_1206
- removed R6, R7, R8, R9: 10K, microbuilder:_1206MP
- removed U2: SHT31-DIS, microbuilder:SHT3X
- added C1: 0.1uF, microbuilder:_1206
- added U1: Si7021-A20, microbuilder:DFN6_3X3_SI
Connections:
- removed net ADDR: R8.1, U2.2
- removed net ALERT: U2.3
- removed net RST: R9.2, U2.6
- new net +3V3: C1.1, CN2.P$12, U1.5
- net GND: now also C1.2, U1.2; no longer C2.2, R8.2, U2.7, U2.8, U2.THERMAL
- net SCL: now also U1.6; no longer R6.1, U2.4
- net SDA: now also U1.1; no longer R7.1, U2.1
- net VDD: no longer C2.1, R6.2, R7.2, R9.1, U2.5
Routing:
- net +3V3: track 0.00 -> 47.9 mm, vias 0 -> 2
- net VDD: track 155.6 -> 111.2 mm
- net GND: track 347.2 -> 316.1 mm, vias 19 -> 18
- net SDA: track 50.3 -> 63.2 mm
- net RST: track 12.5 -> 0.00 mm, vias 2 -> 0
- net SCL: track 52.6 -> 59.4 mm
- net VRED: track 30.2 -> 33.4 mm
- net ADDR: track 3.14 -> 0.00 mm
