File: PCB/aircitizen-m5stack-v2/aircitizen-m5stack-v2.sch (EAGLE design)
At the start: 18 parts, among them CN2 CON_PINHD-2X15, Q3 MOSFET-NCHANNELBSS138, U2 SHT31-DIS, U3 MICS-4514

Commit message: Nouvel version pcb V2
Parts:
- removed C2: 10uF, microbuilder:CAP_CERAMIC_1206
- removed R6, R7, R8, R9: 10K, microbuilder:RESISTOR_1206MP
- removed U2: SHT31-DIS, microbuilder:SHT3X
- added C1: 0.1uF, microbuilder:CAP_CERAMIC_1206
- added U1: Si7021-A20, microbuilder:SI7021-A20
Connections:
- removed net ADDR: R8.1, U2.ADDR
- removed net ALERT: U2.ALERT
- removed net RST: R9.2, U2.NRESET
- new net +3V3: C1.1, CN2.12, U1.VDD
- net GND: now also C1.2, U1.GND; no longer C2.2, R8.2, U2.R(VSS), U2.VSS
- net SCL: now also U1.SCL; no longer R6.1, U2.SCL
- net SDA: now also U1.SDA; no longer R7.1, U2.SDA
- net VDD: no longer C2.1, R6.2, R7.2, R9.1, U2.VDD
Other:
- note removed: "SHT31"
